File: body v1/body v1.kicad_pcb (KiCad board)
At the start: 2 copper layers, 2 parts, among them U1 PCF8574T, X1 XIAO-ESP32-S3-Plus-SMD

Commit message: end schema body
Parts:
- added A1: Conn_01x02, Connector_Molex:Molex_KK-254_AE-6410-02A_1x02_P2.54mm_Vertical, F.Cu at (87.3, 82.9)
- added A2: Conn_01x02, Connector_Molex:Molex_KK-254_AE-6410-02A_1x02_P2.54mm_Vertical, F.Cu at (94.5, 82.9)
- added A3: Conn_01x02, Connector_Molex:Molex_KK-254_AE-6410-02A_1x02_P2.54mm_Vertical, F.Cu at (87.3, 90.7)
- added A4: Conn_01x02, Connector_Molex:Molex_KK-254_AE-6410-02A_1x02_P2.54mm_Vertical, F.Cu at (94.5, 90.7)
- added A5: Conn_01x02, Connector_Molex:Molex_KK-254_AE-6410-02A_1x02_P2.54mm_Vertical, F.Cu at (87.3, 98.6)
- added A6: Conn_01x02, Connector_Molex:Molex_KK-254_AE-6410-02A_1x02_P2.54mm_Vertical, F.Cu at (94.5, 98.6)
- added A7: Conn_01x02, Connector_Molex:Molex_KK-254_AE-6410-02A_1x02_P2.54mm_Vertical, F.Cu at (87.3, 106.4)
- added A8: Conn_01x02, Connector_Molex:Molex_KK-254_AE-6410-02A_1x02_P2.54mm_Vertical, F.Cu at (94.5, 106.4)
- added D4: D_Small, Diode_SMD:D_SMA_Handsoldering, F.Cu at (126.0, 50.9)
- added F1: Fuse_Small, Fuse:Fuseholder_Blade_Mini_Keystone_3568, F.Cu at (112.4, 71.7)
- added H1: M3, MountingHole:MountingHole_3.2mm_M3_Pad_Via, F.Cu at (120.2, 82.9)
- added H2: M3, MountingHole:MountingHole_3.2mm_M3_Pad_Via, F.Cu at (120.2, 90.9)
- added H3: M3, MountingHole:MountingHole_3.2mm_M3_Pad_Via, F.Cu at (120.2, 98.8)
- added H4: M3, MountingHole:MountingHole_3.2mm_M3_Pad_Via, F.Cu at (120.2, 106.8)
- added IC1: Con_I2C, Connector_Molex:Molex_KK-254_AE-6410-04A_1x04_P2.54mm_Vertical, F.Cu at (70.5, 43.2)
- added IC2: Con_I2C, Connector_Molex:Molex_KK-254_AE-6410-04A_1x04_P2.54mm_Vertical, F.Cu at (70.5, 56.0)
- added IC3: Con_I2C, Connector_Molex:Molex_KK-254_AE-6410-04A_1x04_P2.54mm_Vertical, F.Cu at (70.5, 68.8)
- added IC4: Con_I2C, Connector_Molex:Molex_KK-254_AE-6410-04A_1x04_P2.54mm_Vertical, F.Cu at (70.5, 81.6)
- added IC5: Con_I2C, Connector_Molex:Molex_KK-254_AE-6410-04A_1x04_P2.54mm_Vertical, F.Cu at (70.5, 94.4)
- added IC6: Con_I2C, Connector_Molex:Molex_KK-254_AE-6410-04A_1x04_P2.54mm_Vertical, F.Cu at (70.5, 107.2)
- added J1: XT60, Connector_AMASS:AMASS_XT60-M_1x02_P7.20mm_Vertical, F.Cu at (113.8, 64.1)
- added JP1: SolderJumper_2_Open, Jumper:SolderJumper-2_P1.3mm_Open_RoundedPad1.0x1.5mm, F.Cu at (126.3, 100.6)
- added JP2: SolderJumper_2_Open, Jumper:SolderJumper-2_P1.3mm_Open_RoundedPad1.0x1.5mm, F.Cu at (126.3, 104.1)
- added JP3: SolderJumper_2_Open, Jumper:SolderJumper-2_P1.3mm_Open_RoundedPad1.0x1.5mm, F.Cu at (126.3, 107.7)
- added K2: FINDER-36.11, Relay_THT:Relay_SPDT_Finder_36.11, F.Cu at (101.8, 82.9)
- added NP1: driver 1, Connector_IDC:IDC-Header_2x05_P2.54mm_Vertical, F.Cu at (90.3, 42.7)
- added NP2: driver 2, Connector_IDC:IDC-Header_2x05_P2.54mm_Vertical, F.Cu at (102.2, 42.7)
- added NP3: IHM + Lidar, Connector_IDC:IDC-Header_2x05_P2.54mm_Vertical, F.Cu at (114.2, 42.7)
- added R1: R, Resistor_SMD:R_1206_3216Metric_Pad1.30x1.75mm_HandSolder, F.Cu at (127.1, 80.6)
- added R108: 4.7k, Resistor_SMD:R_1206_3216Metric_Pad1.30x1.75mm_HandSolder, F.Cu at (127.1, 93.8)
- added R109: 4.7k, Resistor_SMD:R_1206_3216Metric_Pad1.30x1.75mm_HandSolder, F.Cu at (127.1, 97.1)
- added R2: R, Resistor_SMD:R_1206_3216Metric_Pad1.30x1.75mm_HandSolder, F.Cu at (127.1, 83.9)
- added R3: R, Resistor_SMD:R_1206_3216Metric_Pad1.30x1.75mm_HandSolder, F.Cu at (127.1, 87.2)
- added R4: 4.7k, Resistor_SMD:R_1206_3216Metric_Pad1.30x1.75mm_HandSolder, F.Cu at (127.1, 90.5)
- X1: value XIAO-ESP32-S3-Plus-SMD -> ESP32; footprint XIAO_Series_Footprints:XIAO-ESP32-S3-Plus-SMD -> Yosh Lib:xiao s3+
- moved X1 76.2 mm to (96.0, 68.8), turned to 0 degrees
- moved U1 65.6 mm to (105.8, 105.3)
Connections:
- U1 pad 1: unconnected-(U1-A0-Pad1) -> Net-(JP1-B)
- U1 pad 13: unconnected-(U1-~{INT}-Pad13) -> Net-(U1-~{INT})
- U1 pad 2: unconnected-(U1-A1-Pad2) -> Net-(JP2-B)
- U1 pad 3: unconnected-(U1-A2-Pad3) -> Net-(JP3-B)
- X1 pad 10: unconnected-(X1-GPIO8_A9_D9_MISO-Pad10) -> TEAM SW
- X1 pad 11: unconnected-(X1-GPIO9_A10_D10_MOSI-Pad11) -> PWM
- X1 pad 18: RX 1 -> unconnected-(X1-GPIO41_PDM_DATA_RX1-Pad18)
- X1 pad 19: TX 1 -> unconnected-(X1-GPIO42_PDM_CLK_TX1-Pad19)
- X1 pad 21: unconnected-(X1-GPIO11_DVP_Y8_SPI_MOSI1-Pad21) -> LED
- X1 pad 22: unconnected-(X1-GPIO12_DVP_Y7_SPI_MISO1-Pad22) -> Buzzer
- X1 pad 27: GND -> unconnected-(X1-GND1-Pad27)

Commit message: fin schema
Parts:
- removed A1, A2, A3, A4, A5, A6, A7, A8: Conn_01x02, Connector_Molex:Molex_KK-254_AE-6410-02A_1x02_P2.54mm_Vertical
- removed IC5, IC6: Con_I2C, Connector_Molex:Molex_KK-254_AE-6410-04A_1x04_P2.54mm_Vertical
- removed J1: XT60, Connector_AMASS:AMASS_XT60-M_1x02_P7.20mm_Vertical
- added Bat1: XT60, Connector_AMASS:AMASS_XT60-M_1x02_P7.20mm_Vertical, F.Cu at (77.4, 114.6)
- added C1: 10uf, Capacitor_SMD:C_1206_3216Metric_Pad1.33x1.80mm_HandSolder, F.Cu at (185.2, 80.2)
- added C6: 220uF, Capacitor_THT:CP_Radial_D8.0mm_P3.80mm, F.Cu at (175.5, 83.3)
- added D1: SS14, Diode_SMD:D_SMA, F.Cu at (126.5, 42.2)
- added D2: LED_Small, LED_SMD:LED_1206_3216Metric_Pad1.42x1.75mm_HandSolder, F.Cu at (199.7, 53.2)
- added D3: LED_Small, LED_SMD:LED_1206_3216Metric_Pad1.42x1.75mm_HandSolder, F.Cu at (199.7, 56.6)
- added D5: LED_Small, LED_SMD:LED_1206_3216Metric_Pad1.42x1.75mm_HandSolder, F.Cu at (199.7, 60.0)
- added D6: LED_Small, LED_SMD:LED_1206_3216Metric_Pad1.42x1.75mm_HandSolder, F.Cu at (199.7, 63.4)
- added D8: LED_Small, LED_SMD:LED_1206_3216Metric_Pad1.42x1.75mm_HandSolder, F.Cu at (199.7, 66.8)
- added DRV1: Conn_01x02, Connector_AMASS:AMASS_XT30U-M_1x02_P5.0mm_Vertical, F.Cu at (51.3, 113.1)
- added DRV2: Conn_01x02, Connector_AMASS:AMASS_XT30U-M_1x02_P5.0mm_Vertical, F.Cu at (51.3, 120.3)
- added ICM1: PCF8574T, Package_SO:SOIC-16W_7.5x10.3mm_P1.27mm, F.Cu at (177.5, 46.2)
- added J2: BAU, Connector_Molex:Molex_KK-254_AE-6410-03A_1x03_P2.54mm_Vertical, F.Cu at (162.5, 90.3)
- added L1: Conn_01x04, Connector_Molex:Molex_KK-254_AE-6410-04A_1x04_P2.54mm_Vertical, F.Cu at (74.5, 123.6)
- added L2: Lidar, Connector_AMASS:AMASS_XT30U-M_1x02_P5.0mm_Vertical, F.Cu at (51.3, 127.6)
- added P1: Conn_01x02, Connector_AMASS:AMASS_XT30U-M_1x02_P5.0mm_Vertical, F.Cu at (36.0, 113.0)
- added P10: ~, Connector_AMASS:AMASS_XT30U-M_1x02_P5.0mm_Vertical, F.Cu at (63.6, 127.6)
- added P11: ~, Connector_AMASS:AMASS_XT30U-M_1x02_P5.0mm_Vertical, F.Cu at (63.6, 134.8)
- added P12: ~, Connector_AMASS:AMASS_XT30U-M_1x02_P5.0mm_Vertical, F.Cu at (63.6, 142.1)
- added P2: Conn_01x02, Connector_AMASS:AMASS_XT30U-M_1x02_P5.0mm_Vertical, F.Cu at (36.0, 120.2)
- added P3: Conn_01x02, Connector_AMASS:AMASS_XT30U-M_1x02_P5.0mm_Vertical, F.Cu at (36.0, 127.5)
- added P4: Conn_01x02, Connector_AMASS:AMASS_XT30U-M_1x02_P5.0mm_Vertical, F.Cu at (36.0, 134.8)
- added P5: XT30, Connector_AMASS:AMASS_XT30U-M_1x02_P5.0mm_Vertical, F.Cu at (51.3, 134.8)
- added P6: XT30, Connector_AMASS:AMASS_XT30U-M_1x02_P5.0mm_Vertical, F.Cu at (51.3, 142.1)
- added P7: ~, Connector_AMASS:AMASS_XT30U-M_1x02_P5.0mm_Vertical, F.Cu at (51.3, 149.3)
- added P8: ~, Connector_AMASS:AMASS_XT30U-M_1x02_P5.0mm_Vertical, F.Cu at (63.6, 113.1)
- added P9: ~, Connector_AMASS:AMASS_XT30U-M_1x02_P5.0mm_Vertical, F.Cu at (63.6, 120.3)
- added PS1: TEN_50-2411, TEN 50-2411:CONV_TEN_50-2411, F.Cu at (164.6, 65.0)
- added R10: R_Small, Resistor_SMD:R_1206_3216Metric_Pad1.30x1.75mm_HandSolder, F.Cu at (193.7, 69.7)
- added R11: R_Small, Resistor_SMD:R_1206_3216Metric_Pad1.30x1.75mm_HandSolder, F.Cu at (193.7, 73.0)
- added R5: 4.7k, Resistor_SMD:R_1206_3216Metric_Pad1.30x1.75mm_HandSolder, F.Cu at (193.7, 53.2)
- added R6: 4.7k, Resistor_SMD:R_1206_3216Metric_Pad1.30x1.75mm_HandSolder, F.Cu at (193.7, 56.5)
- added R7: R_Small, Resistor_SMD:R_1206_3216Metric_Pad1.30x1.75mm_HandSolder, F.Cu at (193.7, 59.8)
- added R8: R_Small, Resistor_SMD:R_1206_3216Metric_Pad1.30x1.75mm_HandSolder, F.Cu at (193.7, 63.1)
- added R9: R_Small, Resistor_SMD:R_1206_3216Metric_Pad1.30x1.75mm_HandSolder, F.Cu at (193.7, 66.4)
- added U2: TSR1-2450E, Converter_DCDC:Converter_DCDC_TRACO_TSR1-xxxxE_THT, F.Cu at (138.8, 115.7)
- U1: value PCF8574T -> TSR1-2433E; footprint Package_SO:SOIC-16W_7.5x10.3mm_P1.27mm -> Converter_DCDC:Converter_DCDC_TRACO_TSR1-xxxxE_THT
- moved IC1 188.2 mm to (256.0, 75.5)
- moved IC2 187.3 mm to (256.0, 82.5)
- moved IC3 186.6 mm to (256.0, 89.5)
- moved IC4 186.0 mm to (256.0, 96.5)
- moved X1 123.3 mm to (212.5, 28.5), turned to 90 degrees
- moved NP3 114.9 mm to (228.8, 33.6), turned to 180 degrees
- moved NP1 108.9 mm to (198.8, 33.6), turned to 180 degrees
- moved NP2 86.7 mm to (188.5, 33.6), turned to 180 degrees
- moved U1 42.5 mm to (147.0, 115.7)
Connections:
- net TEAM SW renamed TSW
- IC1 pad 2: SCL -> GND
- IC1 pad 3: SDA -> SCL
- IC1 pad 4: GND -> SDA
- IC2 pad 2: SCL -> GND
- IC2 pad 3: SDA -> SCL
- IC2 pad 4: GND -> SDA
- IC3 pad 2: SCL -> GND
- IC3 pad 3: SDA -> SCL
- IC3 pad 4: GND -> SDA
- IC4 pad 2: SCL -> GND
- IC4 pad 3: SDA -> SCL
- IC4 pad 4: GND -> SDA
- JP1 pad 2: Net-(JP1-B) -> Net-(ICM1-A0)
- JP2 pad 2: Net-(JP2-B) -> Net-(ICM1-A1)
- JP3 pad 2: Net-(JP3-B) -> Net-(ICM1-A2)
- NP1 pad 1: Net-(NP1-Pin_1) -> Net-(ICM1-P0)
- NP1 pad 2: Net-(NP1-Pin_2) -> Net-(ICM1-P1)
- NP1 pad 3: Net-(NP1-Pin_3) -> Net-(ICM1-P2)
- NP1 pad 4: Net-(NP1-Pin_4) -> Net-(ICM1-P3)
- NP2 pad 1: Net-(NP2-Pin_1) -> Net-(ICM1-P4)
- NP2 pad 2: Net-(NP2-Pin_2) -> Net-(ICM1-P5)
- NP2 pad 3: Net-(NP2-Pin_3) -> Net-(ICM1-P6)
- NP2 pad 4: Net-(NP2-Pin_4) -> Net-(ICM1-P7)
- NP3 pad 5: SCL -> LED
- NP3 pad 8: LED -> SCL
- R1 pad 1: Net-(JP1-B) -> Net-(ICM1-A0)
- R2 pad 1: Net-(JP2-B) -> Net-(ICM1-A1)
- R3 pad 1: Net-(JP3-B) -> Net-(ICM1-A2)
- R4 pad 2: Net-(U1-~{INT}) -> Net-(ICM1-~{INT})
- U1 pad 1: Net-(JP1-B) -> +24V
- U1 pad 2: Net-(JP2-B) -> GND
- U1 pad 3: Net-(JP3-B) -> +3.3V
- X1 pad 1: STEP 1 -> DIR 4
- X1 pad 11: PWM -> unconnected-(X1-GPIO9_A10_D10_MOSI-Pad11)
- X1 pad 15: DIR 1 -> DIR 3
- X1 pad 16: DIR 2 -> STEP 3
- X1 pad 17: DIR 3 -> DIR 1
- X1 pad 18: unconnected-(X1-GPIO41_PDM_DATA_RX1-Pad18) -> DOUT-xbee
- X1 pad 19: unconnected-(X1-GPIO42_PDM_CLK_TX1-Pad19) -> DIN-xbee
- X1 pad 2: STEP 2 -> STEP 4
- X1 pad 20: unconnected-(X1-GPIO10_XMCLK_ADC_BAT-Pad20) -> STEP 1
- X1 pad 21: LED -> PWM
- X1 pad 22: Buzzer -> LED
- X1 pad 23: DIR 4 -> En5VP
- X1 pad 3: STEP 3 -> DIR 2
- X1 pad 4: STEP 4 -> STEP 2
Routing:
- net +3V3: track 0.00 -> 84.7 mm
- net GND: track 0.00 -> 49.2 mm
- net SDA: track 0.00 -> 28.2 mm
- net TX: track 0.00 -> 26.8 mm
- net SCL: track 0.00 -> 25.7 mm
- net STEP 4: track 0.00 -> 21.5 mm
- net DIR 4: track 0.00 -> 20.4 mm
- net STEP 3: track 0.00 -> 19.0 mm
- net DIR 3: track 0.00 -> 17.9 mm
- net RX: track 0.00 -> 10.4 mm
- net STEP 1: track 0.00 -> 10.2 mm
- net LED: track 0.00 -> 8.86 mm
- net DIR 2: track 0.00 -> 8.55 mm
- net STEP 2: track 0.00 -> 8.55 mm
- net tir: track 0.00 -> 5.80 mm
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
Commit message: nique
Parts:
- removed R108, R109: 4.7k, Resistor_SMD:R_1206_3216Metric_Pad1.30x1.75mm_HandSolder
- added R20: 4.7k, Resistor_SMD:R_1206_3216Metric_Pad1.30x1.75mm_HandSolder, F.Cu at (194.9, 80.9)
- added R21: 4.7k, Resistor_SMD:R_1206_3216Metric_Pad1.30x1.75mm_HandSolder, F.Cu at (194.9, 84.2)
- moved IC4 126.9 mm to (134.2, 132.3)
- moved IC3 126.7 mm to (134.2, 124.5)
- moved IC2 126.5 mm to (134.2, 116.6)
- moved IC1 126.2 mm to (134.2, 108.8)
- moved D1 104.5 mm to (136.0, 146.4)
- moved D4 100.4 mm to (122.9, 151.2)
- moved D2 100.0 mm to (147.1, 138.3)
- moved D5 100.0 mm to (147.1, 145.1)
- moved D8 100.0 mm to (147.1, 151.9)
- moved D3 100.0 mm to (147.1, 141.7)
- moved D6 100.0 mm to (147.1, 148.5)
- moved R5 95.1 mm to (155.0, 140.1)
- moved C6 89.8 mm to (111.1, 145.9)
- moved C1 86.3 mm to (134.9, 150.3)
- moved F1 84.6 mm to (155.9, 144.2)
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Connections:
- NP1 pad 1: Net-(ICM1-P0) -> Net-(ICM1-P3)
- NP1 pad 2: Net-(ICM1-P1) -> Net-(ICM1-P2)
- NP1 pad 3: Net-(ICM1-P2) -> Net-(ICM1-P1)
- NP1 pad 4: Net-(ICM1-P3) -> Net-(ICM1-P0)
- NP3 pad 7: SDA -> SCL
- NP3 pad 8: SCL -> SDA
- X1 pad 1: DIR 4 -> STEP 3
- X1 pad 15: DIR 3 -> STEP 4
- X1 pad 16: STEP 3 -> DIR 4
- X1 pad 17: DIR 1 -> DIR 2
- X1 pad 2: STEP 4 -> DIR 3
- X1 pad 20: STEP 1 -> STEP 2
- X1 pad 3: DIR 2 -> DIR 1
- X1 pad 4: STEP 2 -> STEP 1
Routing:
- net +3V3: track 84.7 -> 0.00 mm
- net GND: track 49.2 -> 0.00 mm
- net Net-(ICM1-P4): track 0.00 -> 29.9 mm
- net Net-(ICM1-P6): track 0.00 -> 29.3 mm
- net SDA: track 28.2 -> 0.00 mm
- net TX: track 26.8 -> 0.00 mm
- net Net-(ICM1-P5): track 0.00 -> 26.4 mm
- net SCL: track 25.7 -> 0.00 mm
- net Net-(ICM1-P7): track 0.00 -> 25.7 mm
- net Net-(ICM1-P3): track 0.00 -> 24.7 mm
- net Net-(ICM1-P1): track 0.00 -> 24.5 mm
- net Net-(ICM1-P2): track 0.00 -> 21.6 mm
- net Net-(ICM1-P0): track 0.00 -> 21.3 mm
- net DIR 1: track 5.74 -> 17.6 mm
- net DIR 2: track 8.55 -> 19.0 mm
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
Commit message: 11/03
Parts:
- removed P11, P12: ~, Connector_AMASS:AMASS_XT30U-M_1x02_P5.0mm_Vertical
- removed R20, R21: 4.7k, Resistor_SMD:R_1206_3216Metric_Pad1.30x1.75mm_HandSolder
- Bat1, DRV1, DRV2, IC1, IC2, IC3, IC4, ICM1, J2, JP1, JP2, JP3, L1, NP1, NP2, NP3, P5, P6, R1, R2, R3, R4, X1: moved to B.Cu
- L2, P1, P10, P2, P3, P4, P7, P8, P9: footprint Connector_AMASS:AMASS_XT30U-M_1x02_P5.0mm_Vertical -> Connector_Molex:Molex_KK-254_AE-6410-02A_1x02_P2.54mm_Vertical; moved to B.Cu
- moved D1 160.4 mm to (236.8, 21.6), turned to -90 degrees
- moved L1 158.4 mm to (26.1, 24.4)
- moved H1 155.3 mm to (18.0, 24.0)
- moved X1 154.3 mm to (59.0, 33.2)
- moved F1 142.1 mm to (27.6, 83.0)
- moved IC1 136.3 mm to (20.2, 34.0), turned to -90 degrees
- moved IC2 134.4 mm to (28.2, 34.0), turned to -90 degrees
- moved Bat1 133.7 mm to (21.0, 76.0)
- moved IC3 133.4 mm to (36.2, 34.0), turned to -90 degrees
- moved IC4 133.3 mm to (44.2, 34.0), turned to -90 degrees
- moved H2 131.9 mm to (18.0, 95.2)
- moved R3 129.0 mm to (79.5, 28.9), turned to -90 degrees
- moved R2 127.8 mm to (77.0, 28.9), turned to -90 degrees
- moved R1 126.8 mm to (74.5, 28.9), turned to -90 degrees
- moved R4 123.1 mm to (95.6, 29.0), turned to 90 degrees
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Connections:
- D1 pad 2: +5V -> +5VL
- NP3 pad 1: TX -> SDA
- NP3 pad 2: PWM -> TSW
- NP3 pad 3: RX -> SCL
- NP3 pad 4: tir -> LED
- NP3 pad 5: LED -> RX
- NP3 pad 6: TSW -> tir
- NP3 pad 7: SCL -> TX
- NP3 pad 8: SDA -> PWM
Routing:
- net Net-(ICM1-P4): track 29.9 -> 0.00 mm
- net Net-(ICM1-P6): track 29.3 -> 0.00 mm
- net Net-(ICM1-P5): track 26.4 -> 0.00 mm
- net Net-(ICM1-P7): track 25.7 -> 0.00 mm
- net Net-(ICM1-P3): track 24.7 -> 0.00 mm
- net Net-(ICM1-P1): track 24.5 -> 0.00 mm
- net Net-(ICM1-P2): track 21.6 -> 0.00 mm
- net Net-(ICM1-P0): track 21.3 -> 0.00 mm
- net DIR 3: track 19.5 -> 0.00 mm
- net DIR 2: track 19.0 -> 0.00 mm
- net DIR 1: track 17.6 -> 0.00 mm
- net DIR 4: track 17.5 -> 0.00 mm
- net STEP 3: track 16.8 -> 0.00 mm
- net STEP 2: track 16.8 -> 0.00 mm
- net STEP 4: track 15.1 -> 0.00 mm
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Other:
- board outline added: 98 x 79.2 mm

Commit message: routage body
Parts:
- removed D2, D3, D5, D6, D8: LED_Small, LED_SMD:LED_1206_3216Metric_Pad1.42x1.75mm_HandSolder
- added DT1: LED_Small, LED_SMD:LED_1206_3216Metric_Pad1.42x1.75mm_HandSolder, F.Cu at (56.0, 43.3)
- added DT2: LED_Small, LED_SMD:LED_1206_3216Metric_Pad1.42x1.75mm_HandSolder, F.Cu at (58.8, 43.3)
- added DT3: LED_Small, LED_SMD:LED_1206_3216Metric_Pad1.42x1.75mm_HandSolder, F.Cu at (64.2, 43.3)
- added DT4: LED_Small, LED_SMD:LED_1206_3216Metric_Pad1.42x1.75mm_HandSolder, F.Cu at (61.5, 43.3)
- added DT5: LED_Small, LED_SMD:LED_1206_3216Metric_Pad1.42x1.75mm_HandSolder, F.Cu at (67.2, 43.3)
- C1, C6, D1, D4, F1, R5, R6: moved to B.Cu
- moved D1 160.6 mm to (78.3, 47.7)
- moved D4 138.8 mm to (81.3, 102.8), turned to -90 degrees
- moved R10 134.9 mm to (61.5, 49.0), turned to -90 degrees
- moved R7 132.7 mm to (56.0, 49.0), turned to -90 degrees
- moved R8 132.6 mm to (58.8, 49.0), turned to -90 degrees
- moved R9 130.6 mm to (64.2, 49.0), turned to -90 degrees
- moved R11 126.5 mm to (67.2, 49.0), turned to -90 degrees
- moved R5 118.4 mm to (103.2, 78.0), turned to 90 degrees
- moved R6 118.4 mm to (105.7, 78.0), turned to 90 degrees
- moved C1 106.8 mm to (134.5, 43.5), turned to 90 degrees
- moved P7 57.0 mm to (138.5, 86.0)
- moved DRV1 54.0 mm to (131.5, 103.8), turned to 180 degrees
- moved L1 52.9 mm to (72.5, 49.8), turned to 90 degrees
- moved DRV2 52.3 mm to (131.5, 96.2), turned to 180 degrees
- moved P8 48.0 mm to (138.5, 78.0)
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Connections:
- DRV1 pad 1: +24V -> GND
- DRV1 pad 2: GND -> +24V
- DRV2 pad 1: +24V -> GND
- DRV2 pad 2: GND -> +24V
- NP3 pad 1: SDA -> TX
- NP3 pad 2: TSW -> PWM
- NP3 pad 3: SCL -> RX
- NP3 pad 4: LED -> tir
- NP3 pad 5: RX -> LED
- NP3 pad 6: tir -> TSW
- NP3 pad 7: TX -> SDA
- NP3 pad 8: PWM -> SCL
- P7 pad 1: +3.3V -> +3V3
- P8 pad 1: +3.3V -> +3V3
- U1 pad 3: +3.3V -> +3V3
- X1 pad 10: TSW -> PWM
- X1 pad 17: DIR 2 -> STEP 2
- X1 pad 20: STEP 2 -> DIR 2
- X1 pad 21: PWM -> TSW
- X1 pad 22: LED -> tir
- X1 pad 3: DIR 1 -> STEP 1
- X1 pad 4: STEP 1 -> DIR 1
- X1 pad 9: tir -> LED
Routing:
- net +3V3: track 0.00 -> 292.4 mm
- net SDA: track 0.00 -> 133.2 mm, vias 0 -> 3
- net SCL: track 0.00 -> 131.3 mm, vias 0 -> 1
- net +5VL: track 0.00 -> 126.9 mm, vias 0 -> 1
- net +24V: track 0.00 -> 89.5 mm
- net +5VP: track 0.00 -> 76.5 mm
- net GND: track 0.00 -> 71.3 mm, vias 0 -> 173
- net +BATT: track 0.00 -> 70.1 mm, vias 0 -> 2
- net DIR 3: track 0.00 -> 46.3 mm
- net STEP 3: track 0.00 -> 46.3 mm
- net DIR 4: track 0.00 -> 43.2 mm
- net STEP 4: track 0.00 -> 43.2 mm
- net DIN-xbee: track 0.00 -> 40.6 mm
- net En5VP: track 0.00 -> 40.1 mm, vias 0 -> 1
- net DOUT-xbee: track 0.00 -> 38.6 mm
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- added copper zone on F.Cu, net +24V
- added copper zone on F.Cu, net +5VP
- added copper zone on F.Cu, net +BATT
- added copper zone on F.Cu, net /24VD
- added copper zone on B.Cu, net GND
- added copper zone on F.Cu, net GND
Other:
- board size 98 x 79.2 mm -> 98 x 69 mm

Commit message: 16/03
Parts:
- removed K2: FINDER-36.11, Relay_THT:Relay_SPDT_Finder_36.11
- added K1: G2RL-1-E, Relay_THT:Relay_SPDT_Omron_G2RL-1-E, B.Cu at (94.2, 99.5)
- added kibuzzard-69B7FC16: G***, kibuzzard-69B7FC16, F.Cu at (120.7, 49.5)
- added kibuzzard-69B7FC1F: G***, kibuzzard-69B7FC1F, F.Cu at (120.7, 47.0)
- added kibuzzard-69B7FC28: G***, kibuzzard-69B7FC28, F.Cu at (100.3, 47.0)
- added kibuzzard-69B7FC2C: G***, kibuzzard-69B7FC2C, F.Cu at (100.3, 49.5)
- added kibuzzard-69B7FC30: G***, kibuzzard-69B7FC30, F.Cu at (100.3, 52.1)
- added kibuzzard-69B7FC34: G***, kibuzzard-69B7FC34, F.Cu at (100.3, 54.6)
- added kibuzzard-69B7FC3A: G***, kibuzzard-69B7FC3A, F.Cu at (100.3, 55.9)
- added kibuzzard-69B7FC3F: G***, kibuzzard-69B7FC3F, F.Cu at (100.3, 57.1)
- added kibuzzard-69B7FC45: G***, kibuzzard-69B7FC45, F.Cu at (100.3, 58.4)
- added kibuzzard-69B7FC49: G***, kibuzzard-69B7FC49, F.Cu at (100.3, 59.7)
- added kibuzzard-69B7FC4C: G***, kibuzzard-69B7FC4C, F.Cu at (100.3, 61.0)
- added kibuzzard-69B7FC50: G***, kibuzzard-69B7FC50, F.Cu at (100.3, 62.2)
- added kibuzzard-69B7FC58: G***, kibuzzard-69B7FC58, F.Cu at (120.7, 52.1)
- added kibuzzard-69B7FC5D: G***, kibuzzard-69B7FC5D, F.Cu at (120.7, 54.6)
- added kibuzzard-69B7FC64: G***, kibuzzard-69B7FC64, F.Cu at (120.7, 57.1)
- added kibuzzard-69B7FC6B: G***, kibuzzard-69B7FC6B, F.Cu at (120.7, 59.7)
- added kibuzzard-69B7FC71: G***, kibuzzard-69B7FC71, F.Cu at (120.7, 62.2)
- added kibuzzard-69B7FC84: G***, kibuzzard-69B7FC84, F.Cu at (120.7, 50.8)
- added kibuzzard-69B7FC8A: G***, kibuzzard-69B7FC8A, F.Cu at (120.7, 53.3)
- added kibuzzard-69B7FC8F: G***, kibuzzard-69B7FC8F, F.Cu at (120.7, 55.9)
- added kibuzzard-69B7FC95: G***, kibuzzard-69B7FC95, F.Cu at (120.7, 58.4)
- added kibuzzard-69B7FC9A: G***, kibuzzard-69B7FC9A, F.Cu at (120.7, 61.0)
- added kibuzzard-69B7FF72: G***, kibuzzard-69B7FF72, B.Cu at (120.9, 65.1)
- added kibuzzard-69B7FF7A: G***, kibuzzard-69B7FF7A, B.Cu at (135.9, 65.1)
- added kibuzzard-69B7FFCA: G***, kibuzzard-69B7FFCA, B.Cu at (150.9, 65.1)
- added kibuzzard-69B800EA: G***, kibuzzard-69B800EA, B.Cu at (150.9, 68.2)
- added kibuzzard-69B80110: G***, kibuzzard-69B80110, B.Cu at (120.9, 68.2)
- added kibuzzard-69B80117: G***, kibuzzard-69B80117, B.Cu at (135.9, 68.2)
- moved R5 30.4 mm to (133.2, 72.7)
- moved R6 30.4 mm to (135.6, 72.7)
- moved Bat1 25.7 mm to (78.7, 97.4), turned to 180 degrees
- moved U1 24.7 mm to (127.4, 106.3), turned to 180 degrees
- moved U2 24.4 mm to (127.4, 93.8), turned to 180 degrees
- moved P5 21.1 mm to (139.1, 97.6)
- moved P6 21.1 mm to (139.1, 105.1)
- moved C6 20.8 mm to (125.1, 82.2)
- moved C1 19.6 mm to (154.1, 44.9)
- moved D1 19.6 mm to (97.9, 49.1)
- moved DRV1 19.6 mm to (151.1, 105.1)
- moved DRV2 19.6 mm to (151.1, 97.6)
- moved DT1 19.6 mm to (75.6, 44.6)
- moved DT2 19.6 mm to (78.3, 44.6)
- moved DT3 19.6 mm to (83.8, 44.6)
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Routing:
- net GND: track 71.3 -> 213.9 mm, vias 173 -> 138
- net +24V: track 89.5 -> 121.0 mm, vias 0 -> 1
- net +3V3: track 292.4 -> 273.9 mm
- net /24VD: track 9.40 -> 3.40 mm
- net Net-(D4-A): track 19.4 -> 14.1 mm
- net +BATT: track 70.1 -> 66.7 mm, vias 2 -> 1
- net SDA: track 133.2 -> 130.6 mm
- net SCL: track 131.3 -> 128.8 mm
- net +5VL: track 126.9 -> 129.3 mm
- net DIN-xbee: track 40.6 -> 39.9 mm
- net DOUT-xbee: track 38.6 -> 38.0 mm
- net Net-(ICM1-P3): track 18.6 -> 18.0 mm
- net En5VP: vias 1 -> 0
- net +5VP: vias 0 -> 1
- added copper zone on B.Cu, net +BATT
- added copper zone on B.Cu, net /24VD
- removed copper zone on F.Cu, net +BATT
- removed copper zone on F.Cu, net /24VD
