File: body v1/body v1.kicad_pcb (KiCad board)
At the start: 2 copper layers, 98 x 69 mm, 184 parts, among them IC1 Con_I2C, IC2 Con_I2C, IC3 Con_I2C, IC4 Con_I2C, J2 BAU, K1 G2RL-1-E, P1 Conn_01x02, P2 Conn_01x02, P3 Conn_01x02, P4 Conn_01x02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

Commit message: modif + carte pami ninja
Parts:
- added G***: LOGO, LOGO, B.Cu at (128.0, 46.7)
- moved G*** 13.1 mm to (145.2, 32.3)
Routing:
- net GND: vias 137 -> 162

Commit message: end head
Parts:
- added kibuzzard-69C651A2: G***, kibuzzard-69C651A2, B.Cu at (140.8, 87.6)
- moved G*** 1.60 mm to (141.9, 64.3)
- moved G*** 0.90 mm to (134.2, 90.2)
Routing:
- net +5VL: track 129.3 -> 134.7 mm
- net GND: vias 162 -> 168
